Commit message: V2.8

File: autonomousim_description/sensors/rpilidar_a2m8.urdf.xacro (robot description, xacro)
@@ -15,5 +15,5 @@
 				<origin rpy="0 0 0" xyz="0 0 0"/>
 				<geometry>
-					<mesh filename="package://eufs_description/meshes/hokuyo_utm_30lx.dae"/>
+					<mesh filename="package://autonomousim_description/meshes/hokuyo_utm_30lx.dae"/>
 				</geometry>
 			</visual>
